File: av_blocks/sitara-av-blocks.kicad_blocks/SURVEYOR_NODE_A.kicad_block/SURVEYOR_NODE_A.kicad_sch (KiCad schematic)
At the start: 1 part

Commit message: Add TBC register (sitara_av.tbc, av-tbc-register skill, scaffold and template page); larger note text; update Dell, Sync card and Protectli fields
Co-Authored-By: Claude Sonnet 5.5 <noreply@anthropic.com>
Parts:
- SURV1: Mounting VESA or Protectli rack shelf - TBC -> TBC (VESA or shelf); Storage 32 GB eMMC + M.2 slot for NVMe (SSD choice TBC) -> 500 GB NVMe SSD (Kingston NV3), M.2
Changed lines of the file:
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@@
 			)
 		)
-		(property "Storage" "32 GB eMMC + M.2 slot for NVMe (SSD choice TBC)"
+		(property "Storage" "500 GB NVMe SSD (Kingston NV3), M.2"
 			(at 90.17 100.33 0)
 			(hide yes)
@@
 			)
 		)
-		(property "Mounting" "VESA or Protectli rack shelf - TBC"
+		(property "Mounting" "TBC (VESA or shelf)"
 			(at 90.17 100.33 0)
 			(hide yes)
