File: templates/sitara-av-project/sitara-av-project.kicad_sch (KiCad schematic)
At the start: 7 parts

Commit message: Add TBC register (sitara_av.tbc, av-tbc-register skill, scaffold and template page); larger note text; update Dell, Sync card and Protectli fields
Co-Authored-By: Claude Sonnet 5.5 <noreply@anthropic.com>
Parts:
- CPU1: Management AMD DASH; which port carries it TBC -> AMD DASH; suspected on the 1 GbE jack, to be confirmed when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; Mounting (none) -> Dell rail kit 3WF88 / 03W88, 4U
- SYNC1: Lanes x4 assumed (TBC) -> Drawn as x4 for slot accounting. Reportedly uses no PCIe da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; SlotWidth 1 (assumed, TBC) -> 1 (retailer listing; vendor datasheet not found)
Other:
- added sheet To be confirmed (tbc.kicad_sch)
- note added: "Client: 1 Sitara Systems: 1"
- note added: "Full register with owner and expected date: sheet 2."
Changed lines of the file:
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@@
 		(effects
 			(font
-				(size 1.78 1.78)
+				(size 2.29 2.29)
 			)
 			(justify left bottom)
@@
 		(effects
 			(font
-				(size 1.78 1.78)
+				(size 2.29 2.29)
+			)
+			(justify left bottom)
+		)
+	)
+	(text "Client: 1   Sitara Systems: 1"
+		(exclude_from_sim no)
+		(at 24.32 269 0)
+		(effects
+			(font
+				(size 2.29 2.29)
 			)
 			(justify left bottom)
@@
 		(effects
 			(font
-				(size 1.78 1.78)
+				(size 2.29 2.29)
 			)
 			(justify left bottom)
@@
 		(effects
 			(font
-				(size 1.78 1.78)
+				(size 2.29 2.29)
+			)
+			(justify left bottom)
+		)
+	)
+	(text "Full register with owner and expected date: sheet 2."
+		(exclude_from_sim no)
+		(at 24.32 263 0)
+		(effects
+			(font
+				(size 2.29 2.29)
 			)
 			(justify left bottom)
@@
 		(effects
 			(font
-				(size 1.78 1.78)
+				(size 2.29 2.29)
 			)
 			(justify left bottom)
+		)
+	)
+	(text_box "TO BE CONFIRMED (TBC): 2 open"
+		(exclude_from_sim no)
+		(at 20.32 247 0)
+		(size 270 28)
+		(margins 1.8175 1.8175 1.8175 1.8175)
+		(stroke
+			(width 0.2)
+			(type solid)
+		)
+		(fill
+			(type none)
+		)
+		(effects
+			(font
+				(size 2.29 2.29)
+			)
+			(justify left top)
 		)
 	)
@@
 			)
 		)
-		(property "SlotWidth" "1 (assumed, TBC)"
+		(property "SlotWidth" "1 (retailer listing; vendor datasheet not found)"
 			(at 250.19 207.01 0)
 			(hide yes)
@@
 			)
 		)
-		(property "Lanes" "x4 assumed (TBC)"
+		(property "Lanes" "Drawn as x4 for slot accounting. Reportedly uses no PCIe data lines (sync runs over ribbon cables to each GPU), electrical lanes not published"
 			(at 250.19 207.01 0)
 			(hide yes)
@@
 			)
 		)
-		(property "Management" "AMD DASH; which port carries it TBC"
+		(property "Management" "AMD DASH; suspected on the 1 GbE jack, to be confirmed when the unit arrives (Oct 28)"
 			(at 85.09 134.62 0)
 			(hide yes)
@@
 		)
 		(property "FormFactor" "Tower Workstation"
+			(at 85.09 134.62 0)
+			(hide yes)
+			(show_name no)
+			(do_not_autoplace no)
+			(effects
+				(font
+					(size 1.78 1.78)
+				)
+			)
+		)
+		(property "Mounting" "Dell rail kit 3WF88 / 03W88, 4U"
 			(at 85.09 134.62 0)
 			(hide yes)
@@
 				)
 			)
+		)
+	)
+	(sheet
+		(at 350.52 222.25)
+		(size 50.8 20.32)
+		(exclude_from_sim no)
+		(in_bom yes)
+		(on_board yes)
+		(dnp no)
+		(fields_autoplaced yes)
+		(stroke
+			(width 0.25)
+			(type solid)
+		)
+		(fill
+			(color 0 0 0 0)
+		)
+		(property "Sheetname" "To be confirmed"
+			(at 350.52 221.49 0)
+			(show_name no)
+			(do_not_autoplace no)
+			(effects
+				(font
+					(size 2.4 2.4)
+					(bold yes)
+				)
+				(justify left bottom)
+			)
+		)
+		(property "Sheetfile" "tbc.kicad_sch"
+			(at 350.52 243.33 0)
+			(show_name no)
+			(do_not_autoplace no)
+			(effects
+				(font
+					(size 1.78 1.78)
+				)
+				(justify left top)
+			)
+		)
+		(instances
+			(project "sitara-av-project"
+				(path "/6abcf7eb-a459-5bbe-a03c-66e5275de101"
+					(page "2")
+				)
+			)
