File: av_blocks/sitara-av-blocks.kicad_blocks/AUDIO_SCARLETT_2I2_A.kicad_block/AUDIO_SCARLETT_2I2_A.kicad_sch (KiCad schematic)
At the start: 1 part

Commit message: Add power budget helper and PowerW symbol fields; record Dell 7875 C20 inlet and 1350 W maximum
Co-Authored-By: Claude Sonnet 5.5 <noreply@anthropic.com>
Parts:
- AUD1: PowerIncludedIn (none) -> host
Changed lines of the file:
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@@
+			)
+		)
+		(property "PowerIncludedIn" "host"
+			(at 119.38 100.33 0)
+			(hide yes)
+			(show_name no)
+			(do_not_autoplace no)
+			(effects
+				(font
+					(size 1.78 1.78)
+				)
 			)
 		)
